File: hardware/relay.kicad_sch (KiCad schematic)
At the start: 2 parts, among them K1 SANYOU_SRD_Form_C

Commit message: labeling
Other:
- note added: "High Voltage"
- title: (none) -> Relay
Changed lines of the file:
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@@
 (kicad_sch (version 20230121) (generator eeschema)
   (paper "A4")
+  (title_block
+    (title "Relay")
+  )
   (junction (at 85.09 39.37) (diameter 0) (color 0 0 0 0)
   )
@@
     (stroke (width 0) (type default))
   )
-  (wire (pts (xy 85.09 48.26) (xy 85.09 49.53))
-    (stroke (width 0) (type default))
-  )
   (wire (pts (xy 80.01 39.37) (xy 80.01 46.99))
     (stroke (width 0) (type default))
@@
     (stroke (width 0) (type default))
   )
+  (wire (pts (xy 88.9 48.26) (xy 85.09 48.26))
+    (stroke (width 0) (type default))
+  )
   (wire (pts (xy 85.09 39.37) (xy 85.09 40.64))
     (stroke (width 0) (type default))
+  )
+  (rectangle (start 52.07 53.34) (end 101.6 72.39)
+    (stroke (width 0) (type default))
+    (fill (type none))
+  )
+  (text "High Voltage" (at 69.85 68.58 0)
+    (effects (font (size 1.27 1.27)) (justify left bottom))
   )
   (hierarchical_label "NC" (shape output) (at 90.17 59.69 0) (fields_autoplaced)
@@
     )
   )
-  (symbol (lib_id "power:GND") (at 85.09 49.53 0) (unit 1)
+  (symbol (lib_id "power:GND") (at 88.9 48.26 0) (unit 1)
     (in_bom yes) (on_board yes) (dnp no)
-    (property "Reference" "#PWR0104" (at 85.09 55.88 0)
-      (effects (font (size 1.27 1.27)) hide)
-    )
-    (property "Value" "GND" (at 85.09 53.34 0)
+    (property "Reference" "#PWR0104" (at 88.9 54.61 0)
+      (effects (font (size 1.27 1.27)) hide)
+    )
+    (property "Value" "GND" (at 88.9 52.07 0)
       (effects (font (size 1.27 1.27)))
     )
-    (property "Footprint" "" (at 85.09 49.53 0)
-      (effects (font (size 1.27 1.27)) hide)
-    )
-    (property "Datasheet" "" (at 85.09 49.53 0)
-      (effects (font (size 1.27 1.27)) hide)
-    )
+    (property "Footprint" "" (at 88.9 48.26 0)
+      (effects (font (size 1.27 1.27)) hide)
+    )
+    (property "Datasheet" "" (at 88.9 48.26 0)
+      (effects (font (size 1.27 1.27)) hide)
+    )
