File: hardware/temperature_sensors.kicad_sch (KiCad schematic)
At the start: 3 parts, among them J2 Conn_01x03

Commit message: fixed 10K resistor for NTC Thermistor
Parts:
- R8: value 4K7 -> 10K
Changed lines of the file:
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@@
       (effects (font (size 1.27 1.27)) (justify left))
     )
-    (property "Value" "4K7" (at 76.2 69.85 0)
+    (property "Value" "10K" (at 76.2 69.85 0)
       (effects (font (size 1.27 1.27)) (justify left))
     )

Commit message: labeling
Other:
- note added: "NTC 10K"
- note added: "ds18b20"
- title: (none) -> Temperature Sensors
Changed lines of the file:
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@@
 (kicad_sch (version 20230121) (generator eeschema)
   (paper "A4")
+  (title_block
+    (title "Temperature Sensors")
+  )
   (junction (at 60.96 48.26) (diameter 0) (color 0 0 0 0)
   )
@@
     (stroke (width 0) (type default))
   )
+  (rectangle (start 90.17 58.42) (end 115.57 66.04)
+    (stroke (width 0) (type default))
+    (fill (type none))
+  )
+  (rectangle (start 90.17 44.45) (end 115.57 55.88)
+    (stroke (width 0) (type default))
+    (fill (type none))
+  )
+  (text "NTC 10K" (at 99.06 63.5 0)
+    (effects (font (size 1.27 1.27)) (justify left bottom))
+  )
+  (text "ds18b20" (at 99.06 49.53 0)
+    (effects (font (size 1.27 1.27)) (justify left bottom))
+  )
   (hierarchical_label "Data" (shape input) (at 57.15 48.26 180) (fields_autoplaced)
